File: cad/cad.kicad_pcb (KiCad board)
At the start: 2 copper layers, 86 parts, among them SW1 SW_Push, SW10 SW_Push, SW11 ResetSW, SW12 SW_Push, SW13 SW_Push, SW14 SW_Push, SW15 SW_Push, SW16 SW_Push, SW17 SW_Push, SW18 SW_Push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

Commit message: cadでswitchを配置
Parts:
- moved SW4 38.0 mm to (51.8, 70.1)
- moved SW5 34.4 mm to (53.3, 88.6)
- moved SW2 31.8 mm to (29.6, 89.0)
- moved SW3 31.7 mm to (31.6, 108.0)
- moved SW6 29.7 mm to (55.3, 108.1)
- moved SW1 26.5 mm to (32.3, 70.1)
