File: cad/mami-reverse.kicad_sch (KiCad schematic)
At the start: 86 parts, among them SW1 SW_Push, SW10 SW_Push, SW11 SW_Push, SW12 SW_Push, SW13 SW_Push, SW14 SW_Push, SW15 SW_Push, SW16 SW_Push, SW17 SW_Push, SW18 SW_Push, SW19 SW_Push, SW2 SW_Push, SW20 SW_Push, SW21 SW_Push, SW22 SW_Push, SW23 SW_Push, SW24 SW_Push, SW25 SW_Push, SW26 SW_Push, SW27 SW_Push, SW28 SW_Push, SW29 SW_Push, SW3 SW_Push, SW30 SW_Push, SW31 SW_Push, SW32 SW_Push, SW33 SW_Push, SW34 SW_Push, SW35 SW_Push, SW36 SW_Push, SW37 SW_Push, SW38 SW_Push, SW39 SW_Push, SW4 SW_Push, SW40 SW_Push, SW41 SW_Push, SW42 SW_Push, SW43 ResetSW, SW5 SW_Push, SW6 SW_Push, SW7 SW_Push, SW8 SW_Push, SW9 SW_Push, U1 ProMicro

Commit message: cadでswitchを配置
Parts:
- renumbered SW43 to SW11, SW11 to SW12, SW12 to SW13, SW13 to SW14, SW14 to SW15, SW15 to SW16, SW16 to SW17, SW17 to SW18, SW18 to SW19, SW19 to SW20, SW20 to SW21, SW21 to SW22, SW22 to SW23, SW23 to SW24, SW24 to SW25, SW25 to SW26, SW26 to SW27, SW27 to SW28, SW28 to SW29, SW29 to SW30, SW30 to SW31, SW31 to SW32, SW32 to SW33, SW33 to SW34, SW34 to SW35, SW35 to SW36, SW36 to SW37, SW37 to SW38, SW38 to SW39, SW39 to SW40, SW40 to SW41, SW41 to SW42, SW42 to SW43
Connections:
- net col0: now also U1.5 (2/D1/SDA); no longer SW41.1, SW42.1, SW43.1, U1.7 (4/D4)
- net col1: now also U1.6 (3/D0/SCL); no longer SW37.1, SW38.1, SW39.1, SW40.1, U1.8 (5/C6)
- net col2: now also U1.7 (4/D4); no longer SW34.1, SW35.1, SW36.1, U1.9 (6/D7)
- net col3: now also U1.8 (5/C6); no longer SW30.1, SW31.1, SW32.1, SW33.1, U1.10 (7/E6)
- net col4: now also U1.20 (F4/A3); no longer SW27.1, SW28.1, SW29.1, U1.11 (8/B4)
- net col5: now also U1.19 (F5/A2); no longer SW23.1, SW24.1, SW25.1, SW26.1, U1.12 (9/B5)
- net row0: now also D22.1 (K), D26.1 (K), D29.1 (K), D33.1 (K), D36.1 (K), D40.1 (K), U1.9 (6/D7); no longer U1.20 (F4/A3)
- net row1: now also D23.1 (K), D27.1 (K), D30.1 (K), D34.1 (K), D37.1 (K), D41.1 (K), U1.10 (7/E6); no longer U1.19 (F5/A2)
- net row2: now also D24.1 (K), D28.1 (K), D31.1 (K), D35.1 (K), D38.1 (K), D42.1 (K), U1.11 (8/B4)
- net row3: now also D25.1 (K), D32.1 (K), D39.1 (K), U1.12 (9/B5); no longer U1.18 (F6/A1)
- net col11: now reaches U1.13 (B6/10)
- net col11: now also SW41.1, SW42.1, SW43.1
- removed net row4: D22.1 (K), D26.1 (K), D29.1 (K), D33.1 (K), D36.1 (K), D40.1 (K), U1.17 (F7/A0)
- removed net row5: D23.1 (K), D27.1 (K), D30.1 (K), D34.1 (K), D37.1 (K), D41.1 (K), U1.16 (B1/15)
- removed net row6: D24.1 (K), D28.1 (K), D31.1 (K), D35.1 (K), D38.1 (K), D42.1 (K), U1.15 (B3/14)
- removed net row7: D25.1 (K), D32.1 (K), D39.1 (K), U1.14 (B2/16)
- new net col10: SW37.1, SW38.1, SW39.1, SW40.1, U1.14 (B2/16)
- new net col6: SW23.1, SW24.1, SW25.1, SW26.1, U1.18 (F6/A1)
- new net col7: SW27.1, SW28.1, SW29.1, U1.17 (F7/A0)
- new net col8: SW30.1, SW31.1, SW32.1, SW33.1, U1.16 (B1/15)
- new net col9: SW34.1, SW35.1, SW36.1, U1.15 (B3/14)
- no-connect marks 6 -> 3
