File: cad/mami.kicad_pcb (KiCad board)
At the start: 2 copper layers, 86 parts, among them SW1 SW_Push, SW10 SW_Push, SW11 SW_Push, SW12 SW_Push, SW13 SW_Push, SW14 SW_Push, SW15 SW_Push, SW16 SW_Push, SW17 SW_Push, SW18 SW_Push, SW19 SW_Push, SW2 SW_Push, SW20 SW_Push, SW21 SW_Push, SW22 SW_Push, SW23 SW_Push, SW24 SW_Push, SW25 SW_Push, SW26 SW_Push, SW27 SW_Push, SW28 SW_Push, SW29 SW_Push, SW3 SW_Push, SW30 SW_Push, SW31 SW_Push, SW32 SW_Push, SW33 SW_Push, SW34 SW_Push, SW35 SW_Push, SW36 SW_Push, SW37 SW_Push, SW38 SW_Push, SW39 SW_Push, SW4 SW_Push, SW40 SW_Push, SW41 SW_Push, SW42 SW_Push, SW43 ResetSW, SW5 SW_Push, SW6 SW_Push, SW7 SW_Push, SW8 SW_Push, SW9 SW_Push, U1 ProMicro

Commit message: キーキャップ変更 shift->1.25u caps->1u
Parts:
- moved SW42 4.66 mm to (264.3, 102.6)
- moved SW3 4.66 mm to (34.4, 102.5)
- moved SW41 2.40 mm to (268.6, 83.5)
- moved SW2 2.23 mm to (30.0, 83.5)
Changed lines of the file:
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@@
 	(footprint "kbd:keyswitch_cherrymx_hotswap_1u"
 		(layer "F.Cu")
-		(at 271 83.54)
+		(at 268.59625 83.54)
 		(property "Reference" "SW41"
 			(at 0 -7.5 0)
@@
 	(footprint "kbd:keyswitch_cherrymx_hotswap_1u"
 		(layer "F.Cu")
-		(at 29.75 102.54)
+		(at 34.405 102.54)
 		(property "Reference" "SW3"
 			(at 0 -7.5 0)
@@
 	(footprint "kbd:keyswitch_cherrymx_hotswap_1u"
 		(layer "F.Cu")
-		(at 27.75 83.54)
+		(at 29.98375 83.54)
 		(property "Reference" "SW2"
 			(at 0 -7.5 0)
@@
 	(footprint "kbd:keyswitch_cherrymx_hotswap_1u"
 		(layer "F.Cu")
-		(at 269 102.54)
+		(at 264.342 102.58)
 		(property "Reference" "SW42"
 			(at 0 -7.5 0)

Commit message: pcb update
Parts:
- U1: value ProMicro -> ProMicro_r
- moved D40 359.6 mm to (272.4, 56.0)
- moved D41 358.6 mm to (274.4, 75.5)
- moved D42 352.4 mm to (270.4, 94.2)
- moved D37 339.0 mm to (253.3, 56.0)
- moved D38 336.1 mm to (253.1, 75.2)
- moved D39 331.9 mm to (250.8, 94.2)
- moved D33 326.4 mm to (230.5, 54.5), turned to 8 degrees
- moved SW43 323.7 mm to (206.0, 47.5)
- moved D34 323.2 mm to (231.0, 73.8), turned to 8 degrees
- moved D36 318.9 mm to (231.8, 112.0), turned to 8 degrees
- moved D35 318.1 mm to (228.9, 93.2), turned to 8 degrees
- moved D29 303.7 mm to (211.1, 57.2), turned to 8 degrees
- moved D30 301.7 mm to (212.1, 76.0), turned to 8 degrees
- moved D31 297.1 mm to (209.9, 95.8), turned to 8 degrees
- moved D32 296.0 mm to (210.1, 114.8), turned to 8 degrees
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Other:
- board outline added: 269.5 x 1.2 mm

Commit message: symmetric schema update pcb
Parts:
- U1: value ProMicro_r -> ProMicro
Connections:
- U1 pad 10: col3 -> row5
- U1 pad 11: col4 -> row6
- U1 pad 12: col5 -> row7
- U1 pad 13: unconnected-(U1-B6/10-Pad13) -> row3
- U1 pad 14: row7 -> row2
- U1 pad 15: row6 -> row1
- U1 pad 16: row5 -> row0
- U1 pad 17: row4 -> col5
- U1 pad 18: row3 -> col4
- U1 pad 19: row1 -> col3
- U1 pad 20: row0 -> col2
- U1 pad 9: col2 -> row4
Changed lines of the file:
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@@
 			)
 		)
-		(property "Value" "ProMicro_r"
+		(property "Value" "ProMicro"
 			(at -0.1 0.05 90)
 			(layer "F.Fab")
@@
 		(sheetname "/")
 		(sheetfile "cad.kicad_sch")
+		(units
+			(unit
+				(name "A")
+				(pins "1" "2" "3" "4" "5" "6" "7" "8" "9" "10" "11" "12" "24" "23" "22"
+					"21" "20" "19" "18" "17" "16" "15" "14" "13"
+				)
+			)
+		)
 		(attr through_hole)
 		(duplicate_pad_numbers_are_jumpers no)
@@
 			(layers "*.Cu" "B.Mask")
 			(remove_unused_layers no)
-			(net "col2")
+			(net "row4")
 			(pinfunction "6/D7_9")
 			(pintype "bidirectional")
@@
 			(layers "*.Cu" "B.Mask")
 			(remove_unused_layers no)
-			(net "col3")
+			(net "row5")
 			(pinfunction "7/E6_10")
 			(pintype "bidirectional")
@@
 			(layers "*.Cu" "B.Mask")
 			(remove_unused_layers no)
-			(net "col4")
+			(net "row6")
 			(pinfunction "8/B4_11")
 			(pintype "bidirectional")
@@
 			(layers "*.Cu" "B.Mask")
 			(remove_unused_layers no)
-			(net "col5")
+			(net "row7")
 			(pinfunction "9/B5_12")
 			(pintype "bidirectional")
@@
 			(layers "*.Cu" "B.Mask")
 			(remove_unused_layers no)
-			(net "unconnected-(U1-B6{slash}10-Pad13)")
+			(net "row3")
 			(pinfunction "B6/10_13")
-			(pintype "bidirectional+no_connect")
+			(pintype "bidirectional")
 		)
 		(pad "14" thru_hole circle
@@
 			(layers "*.Cu" "B.Mask")
 			(remove_unused_layers no)
-			(net "row7")
+			(net "row2")
 			(pinfunction "B2/16_14")
 			(pintype "bidirectional")
@@
 			(layers "*.Cu" "B.Mask")
 			(remove_unused_layers no)
-			(net "row6")
+			(net "row1")
 			(pinfunction "B3/14_15")
 			(pintype "bidirectional")
@@
 			(layers "*.Cu" "B.Mask")
 			(remove_unused_layers no)
-			(net "row5")
+			(net "row0")
 			(pinfunction "B1/15_16")
 			(pintype "bidirectional")
@@
 			(layers "*.Cu" "B.Mask")
 			(remove_unused_layers no)
-			(net "row4")
+			(net "col5")
 			(pinfunction "F7/A0_17")
 			(pintype "bidirectional")
@@
 			(layers "*.Cu" "B.Mask")
 			(remove_unused_layers no)
-			(net "row3")
+			(net "col4")
 			(pinfunction "F6/A1_18")
 			(pintype "bidirectional")
@@
 			(layers "*.Cu" "B.Mask")
 			(remove_unused_layers no)
-			(net "row1")
+			(net "col3")
 			(pinfunction "F5/A2_19")
 			(pintype "bidirectional")
@@
 			(layers "*.Cu" "B.Mask")
 			(remove_unused_layers no)
-			(net "row0")
+			(net "col2")
 			(pinfunction "F4/A3_20")
 			(pintype "bidirectional")
@@
 	)
 	(group ""
-		(members "26bba0ad-1259-4c20-8ca0-bbbe22d0c1cf" "2c8e5274-9f7e-4c18-b42d-74b082c9ebbc"
-			"7e3b1762-c40e-473e-b731-31f37ddeb1cd" "c13e9b8a-f726-4ec3-ab06-08bf7ee6e159"
-		)
-	)
-	(group ""
-		(members "08696400-f1e4-4e1c-b43b-994e49bb2c5a" "3e4fb591-dd65-43f9-8410-0eaeb50dfa53"
-			"efa77993-f028-4e6e-be9f-4cb1f3a92106"
-		)
-	)
-	(group ""
-		(members "2013a222-d54d-4acc-bed1-dab7a8965a24" "3e336dfe-bc99-48c2-bd98-a728052d3605"
-			"409e5932-ec59-4324-8344-45defc3a6457" "99f9ad64-6e67-4c40-99ce-ab39c0270623"
-		)
-	)
-	(group ""
-		(members "3402fb18-8b9f-4d26-bc39-fc0b496f2e44")
-	)
-	(group ""
-		(members "16feb0ae-c85c-4e76-be81-f2e88505dbb5" "21a6e801-458b-4682-800a-cdec8e5ae010"
-			"253f15a2-e907-4f27-861c-501bcb850ccf" "956eee99-8c02-4c89-a877-443d151d94ac"
-		)
-	)
-	(group ""
-		(members "43dbddb4-4099-435d-97a7-59eecd84e631" "82533b0e-2bdd-4f74-a108-55453b39bd6a"
-			"bc5a6c31-a099-4f11-b8a4-7bd303880050" "c6957c1f-a049-40ce-addf-dc1fb77a262c"
-		)
-	)
-	(group ""
-		(members "31ee5643-105b-4fe0-a464-1ab74040a90d" "5b8b948d-2c4a-490f-b59e-a80a058c6522"
-			"b3345de9-52b4-42bc-a867-8c21e72011b3" "e3f85bb4-2776-4858-820f-f756c7a047e1"
-		)
-	)
-	(group ""
-		(members "92e678f6-6be9-416b-a46b-6b1a3720fa44" "9ec8d110-25c7-4ffa-9308-d119fb02a7d3"
-			"f1adad40-d754-4a1e-90de-422a538e7c7e"
-		)
-	)
-	(group ""
-		(members "051e4c7c-4623-46c9-883b-e88839dbc6d7" "6644cd97-e081-4fc0-8023-ab27cfbd1545"
-			"b029441f-af6a-419b-bb52-ab16a8a3547b" "bdc986a7-0bec-4dec-8797-aba4f1e60c39"
-		)
-	)
-	(group ""

Commit message: drawing edge
Parts:
- moved SW15 7.42 mm to (111.5, 61.4)
- moved SW29 7.42 mm to (207.8, 58.8)
- moved SW37 7.42 mm to (248.3, 56.9)
- moved SW1 7.42 mm to (33.3, 57.2)
- moved SW4 7.42 mm to (52.3, 57.2)
- moved SW40 7.42 mm to (267.3, 57.2)
- moved SW42 7.42 mm to (265.2, 95.2)
- moved D10 7.42 mm to (78.2, 106.1)
- moved D11 7.42 mm to (98.7, 51.4)
- moved D12 7.42 mm to (97.5, 70.4)
- moved D13 7.42 mm to (99.7, 89.9)
- moved D14 7.42 mm to (99.5, 109.1)
- moved D16 7.42 mm to (116.5, 73.1)
- moved D20 7.42 mm to (135.1, 75.6)
- moved D22 7.42 mm to (174.3, 55.1)
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Routing:
- net col5: track 0.00 -> 73.7 mm, vias 0 -> 3
Other:
- board size 269.5 x 1.2 mm -> 258.4 x 86.7 mm

Commit message: make corner round
Other:
- outline, holes or cut-outs redrawn
Changed lines of the file:
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@@
-	)
-	(gr_line
-		(start 61.7 121.65)
-		(end 132.59 131.67)
-		(stroke
-			(width 0.1)
-			(type default)
-		)
-		(layer "F.Paste")
-	)
-	(gr_line
-		(start 62 105)
-		(end 21 105)
-		(stroke
-			(width 0.1)
-			(type default)
-		)
-		(layer "F.Paste")
-	)
-	(gr_line
-		(start 62 122)
-		(end 62 105)
-		(stroke
-			(width 0.1)
-			(type default)
-		)
-		(layer "F.Paste")
-	)
-	(gr_line
-		(start 132.62 131.670962)
-		(end 168 131.64)
-		(stroke
-			(width 0.1)
-			(type default)
-		)
-		(layer "F.Paste")
 	)
 	(gr_line
@@
 	)
 	(gr_line
-		(start 21 45)
-		(end 21 104.71)
+		(start 21 46)
+		(end 21 103.7)
 		(stroke
 			(width 0.05)
@@
 		(layer "Edge.Cuts")
 	)
-	(gr_line
-		(start 21 104.71)
-		(end 61.67 104.74)
-		(stroke
-			(width 0.05)
-			(type default)
-		)
-		(layer "Edge.Cuts")
-	)
-	(gr_line
-		(start 61.67 104.724003)
-		(end 61.67 121.654003)
+	(gr_arc
+		(start 21 46)
+		(mid 21.292893 45.292893)
+		(end 22 45)
+		(stroke
+			(width 0.05)
+			(type default)
+		)
+		(layer "Edge.Cuts")
+	)
+	(gr_arc
+		(start 22 104.71)
+		(mid 21.287983 104.414868)
+		(end 20.999828 103.699998)
+		(stroke
+			(width 0.05)
+			(type default)
+		)
+		(layer "Edge.Cuts")
+	)
+	(gr_line
+		(start 22 104.71)
+		(end 60.7 104.74)
+		(stroke
+			(width 0.05)
+			(type default)
+		)
+		(layer "Edge.Cuts")
+	)
+	(gr_arc
+		(start 60.692893 104.74)
+		(mid 61.4 105.032893)
+		(end 61.692893 105.74)
+		(stroke
+			(width 0.05)
+			(type default)
+		)
+		(layer "Edge.Cuts")
+	)
+	(gr_line
+		(start 61.692893 105.74)
+		(end 61.696368 120.749999)
 		(stroke
 			(width 0.05)
@@
 		(layer "Edge.Cuts")
 	)
-	(gr_line
-		(start 167.97 131.67)
-		(end 238.729228 121.725439)
+	(gr_arc
+		(start 62.451894 121.793941)
+		(mid 61.900819 121.397415)
+		(end 61.696443 120.75)
+		(stroke
+			(width 0.05)
+			(type default)
+		)
+		(layer "Edge.Cuts")
+	)
+	(gr_line
+		(start 132.3 131.625)
+		(end 62.451894 121.793941)
+		(stroke
+			(width 0.05)
+			(type default)
+		)
+		(layer "Edge.Cuts")
+	)
+	(gr_arc
+		(start 132.549911 131.647331)
+		(mid 132.424271 131.643825)
+		(end 132.3 131.625)
+		(stroke
+			(width 0.05)
+			(type default)
+		)
+		(layer "Edge.Cuts")
+	)
+	(gr_line
+		(start 132.55 131.65)
+		(end 167.875 131.65)
+		(stroke
+			(width 0.05)
+			(type default)
+		)
+		(layer "Edge.Cuts")
+	)
+	(gr_arc
+		(start 168.115691 131.629255)
+		(mid 167.99142 131.64808)
+		(end 167.86578 131.651586)
+		(stroke
+			(width 0.05)
+			(type default)
+		)
+		(layer "Edge.Cuts")
+	)
+	(gr_line
+		(start 168.115691 131.629255)
+		(end 238 121.818899)
+		(stroke
+			(width 0.05)
+			(type default)
+		)
+		(layer "Edge.Cuts")
+	)
+	(gr_arc
+		(start 238.72 105.73)
+		(mid 239.014358 105.019358)
+		(end 239.725 104.725)
+		(stroke
+			(width 0.05)
+			(type default)
+		)
+		(layer "Edge.Cuts")
+	)
+	(gr_arc
+		(start 238.73283 120.849894)
+		(mid 238.527331 121.456093)
+		(end 238 121.818899)
+		(stroke
+			(width 0.05)
+			(type default)
+		)
+		(layer "Edge.Cuts")
+	)
+	(gr_line
+		(start 238.73283 120.849894)
+		(end 238.72 105.725)
 		(stroke
 			(width 0.05)
@@
 	)
 	(gr_line
-		(start 238.72 121.66)
-		(end 238.72 104.729989)
-		(stroke
-			(width 0.05)
-			(type solid)
-		)
-		(layer "Edge.Cuts")
-	)
-	(gr_line
-		(start 238.74 104.73)
-		(end 279.35 104.7)
+		(start 239.725 104.725)
+		(end 278.35 104.7)
 		(stroke
 			(width 0.050803)
@@
 	)
 	(gr_line
-		(start 279.32 44.99)
-		(end 21 45)
-		(stroke
-			(width 0.05)
-			(type default)
-		)
-		(layer "Edge.Cuts")
-	)
-	(gr_line
-		(start 279.35 104.7)
-		(end 279.32 44.99)
+		(start 278.3 45)
+		(end 22 45)
+		(stroke
+			(width 0.05)
+			(type default)
+		)
+		(layer "Edge.Cuts")
+	)
+	(gr_arc
+		(start 278.3 45)
+		(mid 279.007107 45.292893)
+		(end 279.3 46)
+		(stroke
+			(width 0.05)
+			(type default)
+		)
+		(layer "Edge.Cuts")
+	)
+	(gr_arc
+		(start 279.35 103.7)
+		(mid 279.055043 104.405043)
+		(end 278.35 104.7)
+		(stroke
+			(width 0.05)
+			(type default)
+		)
+		(layer "Edge.Cuts")
+	)
+	(gr_line
+		(start 279.35 103.7)
+		(end 279.3 46)
 		(stroke
 			(width 0.050803)

Commit message: silicon gasket hole
Parts:
- moved SW43 69.3 mm to (138.2, 50.1), turned to 90 degrees
- moved SW37 59.8 mm to (248.1, 57.2), turned to 0 degrees
- moved D37 59.5 mm to (253.9, 49.0), turned to 0 degrees
- moved D10 57.5 mm to (78.4, 106.1)
- moved SW10 57.5 mm to (72.5, 113.6)
- moved D18 57.1 mm to (135.8, 56.6)
- moved SW18 57.1 mm to (130.2, 64.1)
- moved D36 26.4 mm to (232.2, 104.7), turned to 8 degrees
- moved SW36 26.0 mm to (228.0, 113.7), turned to 8 degrees
- moved D20 19.7 mm to (137.3, 95.2)
- moved SW20 19.7 mm to (131.5, 102.8)
- moved D8 19.7 mm to (78.8, 67.9)
- moved SW8 19.7 mm to (72.9, 75.3)
- moved SW21 19.5 mm to (124.3, 120.9)
- moved D21 19.3 mm to (130.6, 113.2)
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- renumbered D7 to D10, D39 to D36, D36 to D37, D37 to D38, D38 to D39, D8 to D7, D9 to D8, D10 to D9, SW7 to SW10, SW39 to SW36, SW36 to SW37, SW37 to SW38, SW38 to SW39, SW8 to SW7, SW9 to SW8, SW10 to SW9
Connections:
- SW10 pad 1: col1 -> col2
- SW36 pad 1: col1 -> col2
Routing:
- net row0: track 0.00 -> 47.3 mm
- net VCC: track 0.00 -> 1.99 mm, vias 0 -> 1
- net GND: track 0.00 -> 1.41 mm
- net col5: track 73.7 -> 73.0 mm
Other:
- outline, holes or cut-outs redrawn

Commit message: 回路図エディターをbattery有り＋LED有りに変更
Parts:
- added REF**: SW_SPDT_PCM12, Button_Switch_SMD:SW_SPDT_PCM12, F.Cu at (23.9, 94.6)
- added REF**: JST_PH_S2B-PH-K_1x02_P2.00mm_Horizontal, Connector_JST:JST_PH_S2B-PH-K_1x02_P2.00mm_Horizontal, F.Cu at (96.5, 28.6)
Other:
- outline, holes or cut-outs redrawn

Commit message: LED向き変更
Parts:
- removed the REF** at (23.9, 94.6)
- removed the REF** at (96.5, 28.6)
- removed U1: ProMicro, kbd:ProMicro
- added D43: SK6812MINI-E, LED_SMD:LED_SK6812MINI-E_3.2x2.8mm_P1.5mm_ReverseMount, F.Cu at (33.2, 62.0)
- added D44: SK6812MINI-E, LED_SMD:LED_SK6812MINI-E_3.2x2.8mm_P1.5mm_ReverseMount, F.Cu at (3.71, 6.80)
- added D45: SK6812MINI-E, LED_SMD:LED_SK6812MINI-E_3.2x2.8mm_P1.5mm_ReverseMount, F.Cu at (3.71, 11.7)
- added D46: SK6812MINI-E, LED_SMD:LED_SK6812MINI-E_3.2x2.8mm_P1.5mm_ReverseMount, F.Cu at (3.71, 16.5)
- added D47: SK6812MINI-E, LED_SMD:LED_SK6812MINI-E_3.2x2.8mm_P1.5mm_ReverseMount, F.Cu at (3.71, 21.4)
- added D48: SK6812MINI-E, LED_SMD:LED_SK6812MINI-E_3.2x2.8mm_P1.5mm_ReverseMount, F.Cu at (3.71, 26.3)
- added D49: SK6812MINI-E, LED_SMD:LED_SK6812MINI-E_3.2x2.8mm_P1.5mm_ReverseMount, F.Cu at (3.71, 31.2)
- added D50: SK6812MINI-E, LED_SMD:LED_SK6812MINI-E_3.2x2.8mm_P1.5mm_ReverseMount, F.Cu at (3.71, 36.0)
- added D51: SK6812MINI-E, LED_SMD:LED_SK6812MINI-E_3.2x2.8mm_P1.5mm_ReverseMount, F.Cu at (3.71, 40.9)
- added D52: SK6812MINI-E, LED_SMD:LED_SK6812MINI-E_3.2x2.8mm_P1.5mm_ReverseMount, F.Cu at (12.1, 1.94)
- added D53: SK6812MINI-E, LED_SMD:LED_SK6812MINI-E_3.2x2.8mm_P1.5mm_ReverseMount, F.Cu at (12.1, 6.80)
- added D54: SK6812MINI-E, LED_SMD:LED_SK6812MINI-E_3.2x2.8mm_P1.5mm_ReverseMount, F.Cu at (12.1, 11.7)
- added D55: SK6812MINI-E, LED_SMD:LED_SK6812MINI-E_3.2x2.8mm_P1.5mm_ReverseMount, F.Cu at (12.1, 16.5)
- added D56: SK6812MINI-E, LED_SMD:LED_SK6812MINI-E_3.2x2.8mm_P1.5mm_ReverseMount, F.Cu at (12.1, 21.4)
- added D57: SK6812MINI-E, LED_SMD:LED_SK6812MINI-E_3.2x2.8mm_P1.5mm_ReverseMount, F.Cu at (12.1, 26.3)
- added D58: SK6812MINI-E, LED_SMD:LED_SK6812MINI-E_3.2x2.8mm_P1.5mm_ReverseMount, F.Cu at (12.1, 31.2)
- added D59: SK6812MINI-E, LED_SMD:LED_SK6812MINI-E_3.2x2.8mm_P1.5mm_ReverseMount, F.Cu at (12.1, 36.0)
- added D60: SK6812MINI-E, LED_SMD:LED_SK6812MINI-E_3.2x2.8mm_P1.5mm_ReverseMount, F.Cu at (12.1, 40.9)
- added D61: SK6812MINI-E, LED_SMD:LED_SK6812MINI-E_3.2x2.8mm_P1.5mm_ReverseMount, F.Cu at (20.6, 1.94)
- added D62: SK6812MINI-E, LED_SMD:LED_SK6812MINI-E_3.2x2.8mm_P1.5mm_ReverseMount, F.Cu at (20.6, 6.80)
- added D63: SK6812MINI-E, LED_SMD:LED_SK6812MINI-E_3.2x2.8mm_P1.5mm_ReverseMount, F.Cu at (20.6, 11.7)
- added D64: SK6812MINI-E, LED_SMD:LED_SK6812MINI-E_3.2x2.8mm_P1.5mm_ReverseMount, F.Cu at (20.6, 16.5)
- added D65: SK6812MINI-E, LED_SMD:LED_SK6812MINI-E_3.2x2.8mm_P1.5mm_ReverseMount, F.Cu at (20.6, 21.4)
- added D66: SK6812MINI-E, LED_SMD:LED_SK6812MINI-E_3.2x2.8mm_P1.5mm_ReverseMount, F.Cu at (20.6, 26.3)
- added D67: SK6812MINI-E, LED_SMD:LED_SK6812MINI-E_3.2x2.8mm_P1.5mm_ReverseMount, F.Cu at (20.6, 31.2)
- added D68: SK6812MINI-E, LED_SMD:LED_SK6812MINI-E_3.2x2.8mm_P1.5mm_ReverseMount, F.Cu at (20.6, 36.0)
- added D69: SK6812MINI-E, LED_SMD:LED_SK6812MINI-E_3.2x2.8mm_P1.5mm_ReverseMount, F.Cu at (20.6, 40.9)
- added D70: SK6812MINI-E, LED_SMD:LED_SK6812MINI-E_3.2x2.8mm_P1.5mm_ReverseMount, F.Cu at (29.0, 1.94)
- added D71: SK6812MINI-E, LED_SMD:LED_SK6812MINI-E_3.2x2.8mm_P1.5mm_ReverseMount, F.Cu at (29.0, 6.80)
- added D72: SK6812MINI-E, LED_SMD:LED_SK6812MINI-E_3.2x2.8mm_P1.5mm_ReverseMount, F.Cu at (29.0, 11.7)
- added D73: SK6812MINI-E, LED_SMD:LED_SK6812MINI-E_3.2x2.8mm_P1.5mm_ReverseMount, F.Cu at (29.0, 16.5)
- added D74: SK6812MINI-E, LED_SMD:LED_SK6812MINI-E_3.2x2.8mm_P1.5mm_ReverseMount, F.Cu at (29.0, 21.4)
- added D75: SK6812MINI-E, LED_SMD:LED_SK6812MINI-E_3.2x2.8mm_P1.5mm_ReverseMount, F.Cu at (29.0, 26.3)
- added D76: SK6812MINI-E, LED_SMD:LED_SK6812MINI-E_3.2x2.8mm_P1.5mm_ReverseMount, F.Cu at (29.0, 31.2)
- added D77: SK6812MINI-E, LED_SMD:LED_SK6812MINI-E_3.2x2.8mm_P1.5mm_ReverseMount, F.Cu at (29.0, 36.0)
- added D78: SK6812MINI-E, LED_SMD:LED_SK6812MINI-E_3.2x2.8mm_P1.5mm_ReverseMount, F.Cu at (29.0, 40.9)
- added D79: SK6812MINI-E, LED_SMD:LED_SK6812MINI-E_3.2x2.8mm_P1.5mm_ReverseMount, F.Cu at (37.4, 1.94)
- added D80: SK6812MINI-E, LED_SMD:LED_SK6812MINI-E_3.2x2.8mm_P1.5mm_ReverseMount, F.Cu at (37.4, 6.80)
- added D81: SK6812MINI-E, LED_SMD:LED_SK6812MINI-E_3.2x2.8mm_P1.5mm_ReverseMount, F.Cu at (37.4, 11.7)
- added D82: SK6812MINI-E, LED_SMD:LED_SK6812MINI-E_3.2x2.8mm_P1.5mm_ReverseMount, F.Cu at (37.4, 16.5)
- added D83: SK6812MINI-E, LED_SMD:LED_SK6812MINI-E_3.2x2.8mm_P1.5mm_ReverseMount, F.Cu at (37.4, 21.4)
- added D84: SK6812MINI-E, LED_SMD:LED_SK6812MINI-E_3.2x2.8mm_P1.5mm_ReverseMount, F.Cu at (37.4, 26.3)
- added REF**: SuperMini, taku:nano, F.Cu at (143.1, 47.4)
Routing:
- net col5: track 73.0 -> 3.03 mm
- net row0: track 47.3 -> 1.27 mm
