File: cad/mami.kicad_pcb (KiCad board)
At the start: 2 copper layers, 252 x 87.7 mm, 86 parts, among them SW43 ResetSW, U1 Micon_BLEMicroPro

Commit message: 手動配線
Parts:
- added J1: Conn_01x02_Pin, kbd-parts:Battery_BMP_2pin, F.Cu at (161.0, 81.1)
- added L1: SK6812MINI-E, kbd-parts:LED_SK6812MINI-E_BL, F.Cu at (170.6, 83.5)
- added L10: SK6812MINI-E, kbd-parts:LED_SK6812MINI-E_BL, F.Cu at (247.2, 95.3)
- added L11: SK6812MINI-E, kbd-parts:LED_SK6812MINI-E_BL, F.Cu at (227.4, 94.6)
- added L12: SK6812MINI-E, kbd-parts:LED_SK6812MINI-E_BL, F.Cu at (208.6, 97.3)
- added L13: SK6812MINI-E, kbd-parts:LED_SK6812MINI-E_BL, F.Cu at (189.7, 100.0)
- added L14: SK6812MINI-E, kbd-parts:LED_SK6812MINI-E_BL, F.Cu at (170.8, 102.7)
- added L15: SK6812MINI-E, kbd-parts:LED_SK6812MINI-E_BL, F.Cu at (170.7, 121.9)
- added L16: SK6812MINI-E, kbd-parts:LED_SK6812MINI-E_BL, F.Cu at (189.6, 119.3)
- added L17: SK6812MINI-E, kbd-parts:LED_SK6812MINI-E_BL, F.Cu at (208.4, 116.6)
- added L18: SK6812MINI-E, kbd-parts:LED_SK6812MINI-E_BL, F.Cu at (227.3, 113.9)
- added L19: SK6812MINI-E, kbd-parts:LED_SK6812MINI-E_BL, F.Cu at (228.8, 132.9)
- added L2: SK6812MINI-E, kbd-parts:LED_SK6812MINI-E_BL, F.Cu at (189.5, 80.8)
- added L20: SK6812MINI-E, kbd-parts:LED_SK6812MINI-E_BL, F.Cu at (207.6, 135.9)
- added L21: SK6812MINI-E, kbd-parts:LED_SK6812MINI-E_BL, F.Cu at (177.0, 140.3)
- added L22: SK6812MINI-E, kbd-parts:LED_SK6812MINI-E_BL, F.Cu at (123.0, 140.3)
- added L23: SK6812MINI-E, kbd-parts:LED_SK6812MINI-E_BL, F.Cu at (92.4, 135.9)
- added L24: SK6812MINI-E, kbd-parts:LED_SK6812MINI-E_BL, F.Cu at (71.2, 132.9)
- added L25: SK6812MINI-E, kbd-parts:LED_SK6812MINI-E_BL, F.Cu at (72.7, 113.9)
- added L26: SK6812MINI-E, kbd-parts:LED_SK6812MINI-E_BL, F.Cu at (91.6, 116.6)
- added L27: SK6812MINI-E, kbd-parts:LED_SK6812MINI-E_BL, F.Cu at (110.4, 119.3)
- added L28: SK6812MINI-E, kbd-parts:LED_SK6812MINI-E_BL, F.Cu at (129.3, 121.9)
- added L29: SK6812MINI-E, kbd-parts:LED_SK6812MINI-E_BL, F.Cu at (129.2, 102.7)
- added L3: SK6812MINI-E, kbd-parts:LED_SK6812MINI-E_BL, F.Cu at (208.3, 78.1)
- added L30: SK6812MINI-E, kbd-parts:LED_SK6812MINI-E_BL, F.Cu at (110.3, 100.0)
- added L31: SK6812MINI-E, kbd-parts:LED_SK6812MINI-E_BL, F.Cu at (91.4, 97.3)
- added L32: SK6812MINI-E, kbd-parts:LED_SK6812MINI-E_BL, F.Cu at (72.6, 94.6)
- added L33: SK6812MINI-E, kbd-parts:LED_SK6812MINI-E_BL, F.Cu at (52.9, 95.3)
- added L34: SK6812MINI-E, kbd-parts:LED_SK6812MINI-E_BL, F.Cu at (52.9, 114.4)
- added L35: SK6812MINI-E, kbd-parts:LED_SK6812MINI-E_BL, F.Cu at (33.8, 114.4)
- added L36: SK6812MINI-E, kbd-parts:LED_SK6812MINI-E_BL, F.Cu at (33.8, 95.3)
- added L37: SK6812MINI-E, kbd-parts:LED_SK6812MINI-E_BL, F.Cu at (33.8, 76.3)
- added L38: SK6812MINI-E, kbd-parts:LED_SK6812MINI-E_BL, F.Cu at (52.9, 76.3)
- added L39: SK6812MINI-E, kbd-parts:LED_SK6812MINI-E_BL, F.Cu at (72.8, 75.4)
- added L4: SK6812MINI-E, kbd-parts:LED_SK6812MINI-E_BL, F.Cu at (227.2, 75.4)
- added L40: SK6812MINI-E, kbd-parts:LED_SK6812MINI-E_BL, F.Cu at (91.7, 78.1)
- added L41: SK6812MINI-E, kbd-parts:LED_SK6812MINI-E_BL, F.Cu at (110.5, 80.8)
- added L42: SK6812MINI-E, kbd-parts:LED_SK6812MINI-E_BL, F.Cu at (129.4, 83.5)
- added L5: SK6812MINI-E, kbd-parts:LED_SK6812MINI-E_BL, F.Cu at (247.2, 76.3)
- added L6: SK6812MINI-E, kbd-parts:LED_SK6812MINI-E_BL, F.Cu at (266.2, 76.3)
- added L7: SK6812MINI-E, kbd-parts:LED_SK6812MINI-E_BL, F.Cu at (266.2, 95.3)
- added L8: SK6812MINI-E, kbd-parts:LED_SK6812MINI-E_BL, F.Cu at (266.2, 114.4)
- added L9: SK6812MINI-E, kbd-parts:LED_SK6812MINI-E_BL, F.Cu at (247.2, 114.4)
- D1, D10, D11, D12, D13, D14, D15, D16, D17, D18, D19, D2, D20, D21, D22, D23, D24, D25, D26, D27, D28, D29, D3, D30, D31, D32, D33, D34, D35, D36, D37, D38, D39, D4, D40, D41, D42, D5, D6, D7, D8, D9: footprint Diode_SMD:D_SOD-123 -> kbd-parts:Diode_SMD
- moved SW43 28.6 mm to (150.0, 78.8), turned to 0 degrees
- moved D25 25.9 mm to (194.0, 133.7)
- moved D36 19.5 mm to (236.6, 127.2)
- moved D39 19.1 mm to (255.1, 109.7)
- moved D42 18.9 mm to (273.9, 109.7)
- moved D32 18.2 mm to (217.5, 130.1)
- moved D37 15.3 mm to (255.4, 71.6)
- moved D40 14.9 mm to (273.8, 71.6)
- moved D41 14.3 mm to (273.9, 91.0)
- moved D38 14.1 mm to (254.8, 90.9)
- moved D6 9.56 mm to (61.4, 109.5)
- moved D3 9.18 mm to (42.1, 109.2)
- moved D21 8.44 mm to (138.8, 137.6)
- moved D24 5.68 mm to (177.9, 114.9)
- moved D35 5.41 mm to (234.7, 107.2)
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- renumbered ECS to SW1, L_CTRL to SW10, E to SW11, D to SW12, C to SW13, CMD to SW14, R to SW15, F to SW16, V to SW17, T to SW18, G to SW19, TAB to SW2, B to SW20, L_SPACE to SW21, Y to SW22, H to SW23, N to SW24, R_SPACE to SW25, U to SW26, J to SW27, M to SW28, I to SW29, L_SHIFT to SW3, K to SW30, , to SW31, R_CTRL to SW32, O to SW33, L to SW34, DOT to SW35, FN to SW36, P to SW37, COLON to SW38, BLSH to SW39, Q to SW4, BSPC to SW40, ENTER to SW41, R_SHIFT to SW42, A to SW5, Z to SW6, W to SW7, S to SW8, X to SW9
Connections:
- U1 pad 16: row0 -> unconnected-(U1-B1/PIN16-Pad16)
- U1 pad 17: unconnected-(U1-F7/PIN17-Pad17) -> col2
- U1 pad 18: col2 -> col1
- U1 pad 19: col1 -> col0
- U1 pad 20: col0 -> row0
- U1 pad 5: col3 -> row4
- U1 pad 6: col4 -> col3
- U1 pad 7: col5 -> col4
- U1 pad 8: unconnected-(U1-C6/PIN8-Pad8) -> col5
- U1 pad 9: row4 -> unconnected-(U1-D7/PIN9-Pad9)
Routing:
- net GND: track 987.2 -> 634.3 mm, vias 66 -> 29
- net row7: track 201.7 -> 114.6 mm, vias 6 -> 1
- net col2: track 363.7 -> 288.2 mm, vias 16 -> 15
- net reset: track 70.4 -> 4.42 mm, vias 4 -> 0
- net VCC: track 1006.4 -> 1070.8 mm, vias 91 -> 65
- net col5: track 252.8 -> 190.0 mm, vias 13 -> 15
- net row4: track 181.0 -> 121.4 mm, vias 11 -> 3
- net Net-(L21-DOUT): track 0.00 -> 48.9 mm
- net Net-(D63-DOUT): track 48.4 -> 0.00 mm
- net col4: track 154.7 -> 202.7 mm, vias 3 -> 15
- net Net-(D43-DOUT): track 45.1 -> 0.00 mm, vias 6 -> 0
- net Net-(L33-DOUT): track 0.00 -> 44.8 mm, vias 0 -> 2
- net Net-(D1-A): track 47.9 -> 5.14 mm, vias 5 -> 0
- net Net-(D46-DOUT): track 42.3 -> 0.00 mm, vias 4 -> 0
- net Net-(D44-DOUT): track 41.9 -> 0.00 mm, vias 6 -> 0
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Other:
- board size 252 x 87.7 mm -> 252 x 89.2 mm

Commit message: 未接続0
Parts:
- moved D26 0.56 mm to (196.9, 75.1)
- moved D22 0.54 mm to (178.1, 77.9)
- moved D17 0.53 mm to (119.4, 115.8)
- moved D13 0.46 mm to (100.7, 113.2)
- moved D18 0.42 mm to (137.8, 80.0)
- moved D20 0.42 mm to (138.4, 118.6)
- moved D7 0.41 mm to (82.1, 72.2)
- moved D9 0.40 mm to (81.9, 110.5)
- moved D29 0.37 mm to (215.7, 72.3)
- moved D4 0.33 mm to (61.6, 71.7)
- moved D33 0.33 mm to (234.4, 69.7)
Routing:
- net GND: track 634.3 -> 0.45 mm, vias 29 -> 1
- net col5: track 190.0 -> 177.5 mm
- net Net-(L33-DOUT): track 44.8 -> 40.1 mm
- net VCC: track 1070.8 -> 1067.4 mm, vias 65 -> 49
- net row6: track 142.1 -> 139.7 mm
- net Net-(L35-DOUT): track 34.0 -> 32.4 mm
- net row2: track 124.1 -> 122.8 mm, vias 0 -> 2
- net row7: track 114.6 -> 115.5 mm
- net BAT+: track 22.4 -> 23.2 mm
- net Net-(L36-DOUT): track 30.5 -> 29.8 mm
- net row0: track 101.9 -> 101.8 mm, vias 1 -> 0
- added copper zone on B.Cu, net GND
- added copper zone on F.Cu, net GND

Commit message: error 0 git add *
Parts:
- moved D11 0.43 mm to (100.6, 74.7)
- moved D15 0.41 mm to (119.2, 77.4)
- moved D7 0.08 mm to (82.1, 72.1)
Routing:
- net col4: track 202.6 -> 178.4 mm, vias 15 -> 12
- net VCC: track 1067.4 -> 1069.5 mm, vias 49 -> 47
- net Net-(L33-DOUT): track 40.1 -> 40.7 mm
- net row4: track 121.7 -> 121.9 mm, vias 3 -> 2
- net col5: vias 15 -> 14
- net col3: vias 18 -> 16
- net col2: vias 15 -> 14
