File: cad/mami.kicad_pcb (KiCad board)
At the start: 2 copper layers, 252 x 89.2 mm, 129 parts, among them J1 Conn_01x02_Pin, SW1 SW_Push, SW10 SW_Push, SW11 SW_Push, SW12 SW_Push, SW13 SW_Push, SW14 SW_Push, SW15 SW_Push, SW16 SW_Push, SW17 SW_Push, SW18 SW_Push, SW19 SW_Push, SW2 SW_Push, SW20 SW_Push, SW21 SW_Push, SW22 SW_Push, SW23 SW_Push, SW24 SW_Push, SW25 SW_Push, SW26 SW_Push, SW27 SW_Push, SW28 SW_Push, SW29 SW_Push, SW3 SW_Push, SW30 SW_Push, SW31 SW_Push, SW32 SW_Push, SW33 SW_Push, SW34 SW_Push, SW35 SW_Push, SW36 SW_Push, SW37 SW_Push, SW38 SW_Push, SW39 SW_Push, SW4 SW_Push, SW40 SW_Push, SW41 SW_Push, SW42 SW_Push, SW43 ResetSW, SW5 SW_Push, SW6 SW_Push, SW7 SW_Push, SW8 SW_Push, SW9 SW_Push, U1 Micon_BLEMicroPro

Commit message: v3.3
Parts:
- moved D25 11.9 mm to (182.5, 130.8)
- moved D21 11.2 mm to (128.6, 133.0)
- moved D7 5.91 mm to (77.0, 69.2)
- moved D9 5.84 mm to (76.8, 107.7)
- moved D10 5.75 mm to (76.0, 125.6)
- moved D32 5.72 mm to (213.6, 126.0)
- moved SW9 5.70 mm to (68.4, 105.8), turned to -4.4 degrees
- moved SW7 5.69 mm to (68.5, 67.3), turned to -4.4 degrees
- moved D20 5.58 mm to (133.7, 115.6)
- moved SW8 5.56 mm to (68.4, 86.6), turned to -4.4 degrees
- moved SW10 5.47 mm to (67.1, 124.8), turned to -4.4 degrees
- moved SW20 5.46 mm to (125.6, 113.3)
- moved L26 5.46 mm to (87.1, 113.5)
- moved L28 5.46 mm to (124.8, 118.8)
- moved L27 5.46 mm to (105.9, 116.2)
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Routing:
- net VCC: track 1069.5 -> 1110.1 mm, vias 47 -> 37
- net col2: track 288.2 -> 306.2 mm, vias 14 -> 15
- net Net-(D25-A): track 13.1 -> 5.38 mm
- net col3: track 258.8 -> 265.2 mm
- net Net-(D21-A): track 10.4 -> 4.81 mm
- net BAT+: track 23.0 -> 27.5 mm, vias 0 -> 1
- net row4: track 121.9 -> 117.9 mm, vias 2 -> 0
- net col4: track 178.4 -> 174.4 mm, vias 12 -> 11
- net row3: track 98.4 -> 102.3 mm
- net row7: track 115.5 -> 118.2 mm
- net Net-(L36-DOUT): track 29.8 -> 27.1 mm
- net Net-(L7-DOUT): track 39.2 -> 36.5 mm
- net col5: track 177.5 -> 175.1 mm, vias 14 -> 15
- net LED: track 18.9 -> 21.1 mm, vias 1 -> 2
- net Net-(L32-DOUT): track 16.0 -> 14.2 mm
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Other:
- board size 252 x 89.2 mm -> 251.8 x 87.8 mm
- board text added: "Authored by T.MORI"
- board text removed: "Authored by t.mori"
